Commit message: fix the mesh orientation

File: nikita_description/urdf/mesh_leg.xacro (robot description, xacro)
@@ -50,5 +50,7 @@
     <link name="${prefix}_tibia_link">
       <visual>
-        <origin xyz="-0.015 0.04 0" rpy="${-90 * pi / 180} ${90 * pi / 180} ${180 * pi / 180}"/>
+        <!-- Rotate the CAD mesh by 90 degrees about the servo axis (link X),
+             including its offset from that axis, to match assembly_complete.py. -->
+        <origin xyz="-0.015 0 0.04" rpy="${-180 * pi / 180} 0 ${90 * pi / 180}"/>
         <geometry><mesh filename="package://nikita_description/meshes/assembly_tibia.stl" scale="${mesh_scale}"/></geometry>
         <material name="light_blue"/>

File: nikita_description/urdf/nikita_mesh.urdf.xacro (robot description, xacro)
@@ -24,9 +24,36 @@
   <xacro:mesh_hexapod_leg prefix="left_mid" cx="0.000" cy="-0.088" psi_deg="-90.0"/>
   <xacro:mesh_hexapod_leg prefix="left_back" cx="-0.109" cy="-0.068" psi_deg="-135.0"/>
-  <!-- Controller-compatible head joints.  The mesh model intentionally has
-       no head visual or collision geometry. -->
-  <joint name="head_yaw_joint" type="revolute"><parent link="base_link"/><child link="head_yaw_link"/><origin xyz="0.130 0 ${coxa_height}"/><axis xyz="0 0 1"/><limit lower="${-30*pi/180}" upper="${30*pi/180}" effort="1.5" velocity="4.0"/></joint>
-  <link name="head_yaw_link"><inertial><mass value="0.001"/><inertia ixx="1e-8" ixy="0" ixz="0" iyy="1e-8" iyz="0" izz="1e-8"/></inertial></link>
-  <joint name="head_pitch_joint" type="revolute"><parent link="head_yaw_link"/><child link="head_pitch_link"/><origin xyz="0 0 0.020"/><axis xyz="0 1 0"/><limit lower="${-20*pi/180}" upper="${20*pi/180}" effort="1.5" velocity="4.0"/></joint>
-  <link name="head_pitch_link"><inertial><mass value="0.001"/><inertia ixx="1e-8" ixy="0" ixz="0" iyy="1e-8" iyz="0" izz="1e-8"/></inertial></link>
+  <!-- Head transforms reproduce the zero-angle placement in
+       cad/assembly_complete.py.  The body mesh already contains the yaw
+       servo; these links add its coxa bracket and the pitch-mounted head. -->
+  <joint name="head_yaw_joint" type="revolute">
+    <parent link="base_link"/>
+    <child link="head_yaw_link"/>
+    <origin xyz="0.140175 0 0.04825"/>
+    <axis xyz="0 0 -1"/>
+    <limit lower="${-30*pi/180}" upper="${30*pi/180}" effort="1.5" velocity="4.0"/>
+  </joint>
+  <link name="head_yaw_link">
+    <visual>
+      <origin xyz="0.0295 0 -0.0143" rpy="${90*pi/180} 0 ${-90*pi/180}"/>
+      <geometry><mesh filename="package://nikita_description/meshes/assembly_coxa.stl" scale="0.001 0.001 0.001"/></geometry>
+      <material name="dark_gray"/>
+    </visual>
+    <inertial><mass value="0.001"/><inertia ixx="1e-8" ixy="0" ixz="0" iyy="1e-8" iyz="0" izz="1e-8"/></inertial>
+  </link>
+  <joint name="head_pitch_joint" type="revolute">
+    <parent link="head_yaw_link"/>
+    <child link="head_pitch_link"/>
+    <origin xyz="0.05313138535886 0.0143 -0.00338993770857"/>
+    <axis xyz="0 -1 0"/>
+    <limit lower="${-20*pi/180}" upper="${20*pi/180}" effort="1.5" velocity="4.0"/>
+  </joint>
+  <link name="head_pitch_link">
+    <visual>
+      <origin xyz="0 0 0.035" rpy="${180*pi/180} 0 0"/>
+      <geometry><mesh filename="package://nikita_description/meshes/assembly_head.stl" scale="0.001 0.001 0.001"/></geometry>
+      <material name="dark_gray"/>
+    </visual>
+    <inertial><mass value="0.001"/><inertia ixx="1e-8" ixy="0" ixz="0" iyy="1e-8" iyz="0" izz="1e-8"/></inertial>
+  </link>
 </robot>
