Commit message: fix the colors for nira

File: rumblex_description/urdf/materials.xacro (robot description, xacro)
@@ -3,4 +3,7 @@
   <material name="dark_gray">
     <color rgba="0.3 0.3 0.3 1.0"/>
+  </material>
+  <material name="creamy_white">
+    <color rgba="0.94 0.91 0.82 1.0"/>
   </material>
   <material name="orange">

File: rumblex_description/urdf/nira_model.xacro (robot description, xacro)
@@ -13,5 +13,5 @@
        Collision boxes are CAD envelopes. Masses, limits and dynamics are
        provisional estimates, not measured Nira hardware parameters. -->
-  <xacro:macro name="nira_link" params="name mesh xyz rpy center size mass meshes">
+  <xacro:macro name="nira_link" params="name mesh xyz rpy center size mass meshes material">
     <xacro:property name="dims" value="${[float(v) for v in size.split()]}"/>
     <link name="${name}">
@@ -26,5 +26,5 @@
           <geometry><box size="${size}"/></geometry>
         </xacro:unless>
-        <material name="dark_gray"/>
+        <material name="${material}"/>
       </visual>
       <collision>
@@ -56,5 +56,5 @@
                      xyz="0.0295 0 0.0185" rpy="-1.57079632679 0 1.57079632679"
                      center="0.0265656926794 0 0.0170032120995" size="0.0781313853589 0.041 0.043993575801"
-                     mass="0.12" meshes="${meshes}"/>
+                     mass="0.12" meshes="${meshes}" material="dark_gray"/>
     <xacro:nira_joint name="${prefix}_femur_joint" parent="${prefix}_coxa_link" child="${prefix}_femur_link"
                       xyz="0.0531313853589 -0.0185 0.00750642419903" rpy="1.57079632679 -0.510488321917 3.14159265359" axis="0 0 -1" lower="-30" upper="90"/>
@@ -62,5 +62,5 @@
                      xyz="-0.035 0 0.00425" rpy="1.57079632679 0 1.57079632679"
                      center="-0.0323906817215 0.00458043191449 0.0182498422486" size="0.0847813634429 0.0378201245829 0.0410000000001"
-                     mass="0.12" meshes="${meshes}"/>
+                     mass="0.12" meshes="${meshes}" material="dark_gray"/>
     <xacro:nira_joint name="${prefix}_tibia_joint" parent="${prefix}_femur_link" child="${prefix}_tibia_link"
                       xyz="-0.0622813634428 0.0109904942059 0.0367498422486" rpy="-3.14159265359 0 2.63110433167" axis="0 0 -1" lower="-90" upper="90"/>
@@ -68,5 +68,5 @@
                      xyz="-0.035 0 0.00425" rpy="1.57079632679 0 1.57079632679"
                      center="0.0187125 0.03775 0.0185" size="0.057425 0.114 0.037"
-                     mass="0.1" meshes="${meshes}"/>
+                     mass="0.1" meshes="${meshes}" material="creamy_white"/>
     <!-- Frame at the centre of the CAD rubber toe; its solid is in the tibia mesh. -->
     <joint name="${prefix}_foot_joint" type="fixed">
@@ -87,5 +87,5 @@
     <!-- Coarse body envelope includes the layered chassis and mounted electronics. -->
     <xacro:nira_link name="base_link" mesh="assembly_torso_servo" xyz="0 0 0" rpy="0 0 0"
-                     center="0 0 0.05" size="0.270 0.190 0.110" mass="0.8" meshes="${meshes}"/>
+                     center="0 0 0.05" size="0.270 0.190 0.110" mass="0.8" meshes="${meshes}" material="creamy_white"/>
     <xacro:nira_leg prefix="right_front" xyz="0.11476587931 0.0697658793104 0.0525" rpy="3.14159265359 0 0.785398163397" meshes="${meshes}"/>
     <xacro:nira_leg prefix="right_mid" xyz="0 0.095175 0.0525" rpy="3.14159265359 0 1.57079632679" meshes="${meshes}"/>
@@ -99,5 +99,5 @@
                      xyz="0.0295 0 0.0185" rpy="-1.57079632679 0 1.57079632679"
                      center="0.0265656926794 0 0.0170032120995" size="0.0781313853589 0.041 0.043993575801"
-                     mass="0.12" meshes="${meshes}"/>
+                     mass="0.12" meshes="${meshes}" material="dark_gray"/>
     <xacro:nira_joint name="head_pitch_joint" parent="head_yaw_link" child="head_pitch_link"
                       xyz="0.0531313853589 -0.0185 0.00750642419903" rpy="1.57079632679 -1.55768587311 -3.14159265359" axis="0 0 -1" lower="-20" upper="20"/>
@@ -105,5 +105,5 @@
                      xyz="-0.035 0 0.00425" rpy="1.57079632679 0 1.57079632679"
                      center="-0.0122000005383 0.0226182043846 0.0187537674652" size="0.054 0.0702364087692 0.07"
-                     mass="0.15" meshes="${meshes}"/>
+                     mass="0.15" meshes="${meshes}" material="dark_gray"/>
     <!-- T-mini scan centre: assembly_torso + lidar_ydlidar_tmini.SCAN_HEIGHT.
          The sensor housing is already included in the torso mesh. -->
