Commit message: adapt meshes to new generated stl files

File: rumblex_description/urdf/mesh_leg.xacro (robot description, xacro)
@@ -21,5 +21,5 @@
       <visual>
         <origin xyz="0 0.035 -0.01" rpy="${pi / 2.0} 0 0"/>
-        <geometry><mesh filename="package://rumblex_description/meshes/assembly_coxa.stl" scale="${mesh_scale}"/></geometry>
+        <geometry><mesh filename="${mesh_directory}/assembly_coxa.stl" scale="${mesh_scale}"/></geometry>
         <material name="orange"/>
       </visual>
@@ -35,6 +35,8 @@
     <link name="${prefix}_femur_link">
       <visual>
-        <origin xyz="0.015 0.043 0" rpy="${-90 * pi / 180} ${-90 * pi / 180} ${180 * pi / 180}"/>
-        <geometry><mesh filename="package://rumblex_description/meshes/assembly_femur.stl" scale="${mesh_scale}"/></geometry>
+        <!-- Roll 180 degrees about the leg segment's length axis (link Y),
+             rotating the CAD registration offset about that axis as well. -->
+        <origin xyz="-0.015 0.043 0" rpy="${pi / 2.0} ${pi / 2.0} 0"/>
+        <geometry><mesh filename="${mesh_directory}/assembly_femur.stl" scale="${mesh_scale}"/></geometry>
         <material name="dark_blue"/>
       </visual>
@@ -50,8 +52,8 @@
     <link name="${prefix}_tibia_link">
       <visual>
-        <!-- Rotate the CAD mesh by 90 degrees about the servo axis (link X),
-             including its offset from that axis, to match assembly_complete.py. -->
-        <origin xyz="-0.015 0 0.04" rpy="${-180 * pi / 180} 0 ${90 * pi / 180}"/>
-        <geometry><mesh filename="package://rumblex_description/meshes/assembly_tibia.stl" scale="${mesh_scale}"/></geometry>
+        <!-- Roll 180 degrees about the leg segment's length axis (link Y),
+             including the CAD offset, after the servo-axis registration. -->
+        <origin xyz="0.015 0 -0.04" rpy="0 0 ${pi / 2.0}"/>
+        <geometry><mesh filename="${mesh_directory}/assembly_tibia.stl" scale="${mesh_scale}"/></geometry>
         <material name="light_blue"/>
       </visual>

File: rumblex_description/urdf/nox_mesh.urdf.xacro (robot description, xacro)
@@ -4,4 +4,5 @@
   <xacro:include filename="$(find rumblex_description)/urdf/mesh_leg.xacro"/>
   <xacro:include filename="$(find rumblex_description)/urdf/ros2_control.xacro"/>
+  <xacro:property name="mesh_directory" value="package://rumblex_description/meshes/nox"/>
   <xacro:property name="coxa_length" value="0.050"/>
   <xacro:property name="femur_length" value="0.063"/>
@@ -14,5 +15,5 @@
   </xacro:if>
   <link name="base_link">
-    <visual><origin xyz="0 0 0"/><geometry><mesh filename="package://rumblex_description/meshes/assembly_body_servo.stl" scale="0.001 0.001 0.001"/></geometry><material name="dark_gray"/></visual>
+    <visual><origin xyz="0 0 0"/><geometry><mesh filename="${mesh_directory}/assembly_body_servo.stl" scale="0.001 0.001 0.001"/></geometry><material name="dark_gray"/></visual>
     <collision><origin xyz="0 0 0.020"/><geometry><box size="0.240 0.180 0.025"/></geometry></collision>
     <inertial><origin xyz="0 0 0.045"/><mass value="0.80"/><inertia ixx="0.003" ixy="0" ixz="0" iyy="0.004" iyz="0" izz="0.005"/></inertial>
@@ -37,5 +38,5 @@
     <visual>
       <origin xyz="0.0295 0 -0.0143" rpy="${90*pi/180} 0 ${-90*pi/180}"/>
-      <geometry><mesh filename="package://rumblex_description/meshes/assembly_coxa.stl" scale="0.001 0.001 0.001"/></geometry>
+      <geometry><mesh filename="${mesh_directory}/assembly_coxa.stl" scale="0.001 0.001 0.001"/></geometry>
       <material name="dark_gray"/>
     </visual>
@@ -52,5 +53,5 @@
     <visual>
       <origin xyz="0 0 0.035" rpy="${180*pi/180} 0 0"/>
-      <geometry><mesh filename="package://rumblex_description/meshes/assembly_head.stl" scale="0.001 0.001 0.001"/></geometry>
+      <geometry><mesh filename="${mesh_directory}/assembly_head.stl" scale="0.001 0.001 0.001"/></geometry>
       <material name="dark_gray"/>
     </visual>

Commit message: fix nox mesh joints

File: rumblex_description/urdf/mesh_leg.xacro (robot description, xacro)
@@ -1,18 +1,17 @@
 <?xml version="1.0"?>
 <robot xmlns:xacro="http://www.ros.org/wiki/xacro">
-  <!--
-    Mesh leg variant.  The CAD exports are in millimetres and use the
-    assembly joint as their local reference.  The small origins below are
-    deliberately explicit: they document the CAD-to-URDF registration and
-    keep the joint frames identical to leg.xacro.
-  -->
+  <!-- Nox CAD registration (cad/robot_nox), metres and radians.
+       Joint frames are the horn mounting faces, not the simplified IK frames
+       in leg.xacro. Zero pose matches assembly_complete: CAD angles 0/0/180.
+       Positive joint angles increase the CAD connection angles. The STL
+       exports already contain the femur and tibia rolls; do not apply again. -->
   <xacro:macro name="mesh_hexapod_leg" params="prefix cx cy psi_deg">
-    <xacro:property name="mount_yaw" value="${psi_deg * pi / 180.0 - pi / 2.0}"/>
+    <xacro:property name="mount_yaw" value="${psi_deg * pi / 180.0}"/>
     <xacro:property name="mesh_scale" value="0.001 0.001 0.001"/>
     <joint name="${prefix}_coxa_joint" type="revolute">
       <parent link="base_link"/>
       <child link="${prefix}_coxa_link"/>
-      <origin xyz="${cx} ${cy} ${coxa_height}" rpy="0 0 ${mount_yaw}"/>
-      <axis xyz="0 0 -1"/>
+      <origin xyz="${cx} ${cy} ${coxa_height}" rpy="${pi} 0 ${mount_yaw}"/>
+      <axis xyz="0 0 1"/>
       <limit lower="${-60 * pi / 180}" upper="${60 * pi / 180}" effort="3.0" velocity="6.0"/>
       <dynamics damping="0.1" friction="0.05"/>
@@ -20,14 +19,14 @@
     <link name="${prefix}_coxa_link">
       <visual>
-        <origin xyz="0 0.035 -0.01" rpy="${pi / 2.0} 0 0"/>
+        <origin xyz="0.0295 0 0.0185" rpy="${-pi / 2} 0 ${pi / 2}"/>
         <geometry><mesh filename="${mesh_directory}/assembly_coxa.stl" scale="${mesh_scale}"/></geometry>
         <material name="orange"/>
       </visual>
-      <collision><origin xyz="0 ${coxa_length / 2.0} 0" rpy="${pi / 2.0} 0 0"/><geometry><box size="0.030 0.050 0.045"/></geometry></collision>
-      <inertial><origin xyz="0 ${coxa_length / 2.0} 0"/><mass value="0.12"/><inertia ixx="3.0e-05" ixy="0" ixz="0" iyy="3.0e-05" iyz="0" izz="3.0e-05"/></inertial>
+      <collision><origin xyz="0.0265656926794 0 0.0170032120995"/><geometry><box size="0.0781313853589 0.041 0.043993575801"/></geometry></collision>
+      <inertial><origin xyz="0.0265656926794 0 0.0170032120995"/><mass value="0.12"/><inertia ixx="3.0e-05" ixy="0" ixz="0" iyy="3.0e-05" iyz="0" izz="3.0e-05"/></inertial>
     </link>
     <joint name="${prefix}_femur_joint" type="revolute">
       <parent link="${prefix}_coxa_link"/><child link="${prefix}_femur_link"/>
-      <origin xyz="0 ${coxa_length} 0" rpy="${30 * pi / 180} 0 0"/><axis xyz="1 0 0"/>
+      <origin xyz="0.053131385358869 -0.0185 0.0075064241990335" rpy="${pi / 2} -0.51048832191678 ${pi}"/><axis xyz="0 0 -1"/>
       <limit lower="${-30 * pi / 180}" upper="${90 * pi / 180}" effort="3.0" velocity="6.0"/>
       <dynamics damping="0.1" friction="0.05"/>
@@ -35,16 +34,14 @@
     <link name="${prefix}_femur_link">
       <visual>
-        <!-- Roll 180 degrees about the leg segment's length axis (link Y),
-             rotating the CAD registration offset about that axis as well. -->
-        <origin xyz="-0.015 0.043 0" rpy="${pi / 2.0} ${pi / 2.0} 0"/>
+        <origin xyz="-0.035 0 0.00425" rpy="${pi / 2} 0 ${pi / 2}"/>
         <geometry><mesh filename="${mesh_directory}/assembly_femur.stl" scale="${mesh_scale}"/></geometry>
         <material name="dark_blue"/>
       </visual>
-      <collision><origin xyz="0 ${femur_length / 2.0} 0" rpy="${-pi / 2.0} 0 0"/><geometry><box size="0.030 0.063 0.045"/></geometry></collision>
-      <inertial><origin xyz="0 ${femur_length / 2.0} 0"/><mass value="0.12"/><inertia ixx="4.0e-05" ixy="0" ixz="0" iyy="4.0e-05" iyz="0" izz="4.0e-05"/></inertial>
+      <collision><origin xyz="-0.0325302233968 0.00458351350954 0.0185"/><geometry><box size="0.0850604467937 0.0378201245829 0.041"/></geometry></collision>
+      <inertial><origin xyz="-0.0325302233968 0.00458351350954 0.0185"/><mass value="0.12"/><inertia ixx="4.0e-05" ixy="0" ixz="0" iyy="4.0e-05" iyz="0" izz="4.0e-05"/></inertial>
     </link>
     <joint name="${prefix}_tibia_joint" type="revolute">
       <parent link="${prefix}_femur_link"/><child link="${prefix}_tibia_link"/>
-      <origin xyz="0 ${femur_length} 0" rpy="${-120 * pi / 180} 0 0"/><axis xyz="1 0 0"/>
+      <origin xyz="-0.062560446793669 0.010993575800966 0.037" rpy="${-pi} 0 2.631104331673"/><axis xyz="0 0 -1"/>
       <limit lower="${-90 * pi / 180}" upper="${90 * pi / 180}" effort="3.0" velocity="6.0"/>
       <dynamics damping="0.1" friction="0.05"/>
@@ -52,16 +49,13 @@
     <link name="${prefix}_tibia_link">
       <visual>
-        <!-- Roll 180 degrees about the leg segment's length axis (link Y),
-             including the CAD offset, after the servo-axis registration. -->
-        <origin xyz="0.015 0 -0.04" rpy="0 0 ${pi / 2.0}"/>
+        <origin xyz="-0.035 0 0.00425" rpy="${pi / 2} 0 ${pi / 2}"/>
         <geometry><mesh filename="${mesh_directory}/assembly_tibia.stl" scale="${mesh_scale}"/></geometry>
         <material name="light_blue"/>
       </visual>
-      <collision><origin xyz="0 ${tibia_length / 2.0} 0" rpy="${-pi / 2.0} 0 0"/><geometry><box size="0.025 0.099 0.040"/></geometry></collision>
-      <inertial><origin xyz="0 ${tibia_length / 2.0} 0"/><mass value="0.10"/><inertia ixx="4.0e-05" ixy="0" ixz="0" iyy="4.0e-05" iyz="0" izz="4.0e-05"/></inertial>
+      <collision><origin xyz="0.0179625 0.03775 0.0185"/><geometry><box size="0.055925 0.114 0.037"/></geometry></collision>
+      <inertial><origin xyz="0.0179625 0.03775 0.0185"/><mass value="0.10"/><inertia ixx="4.0e-05" ixy="0" ixz="0" iyy="4.0e-05" iyz="0" izz="4.0e-05"/></inertial>
     </link>
-    <joint name="${prefix}_foot_joint" type="fixed"><parent link="${prefix}_tibia_link"/><child link="${prefix}_foot"/><origin xyz="0 ${tibia_length} 0"/></joint>
+    <joint name="${prefix}_foot_joint" type="fixed"><parent link="${prefix}_tibia_link"/><child link="${prefix}_foot"/><origin xyz="0.028425 0.09225 0.01825" rpy="${-pi / 2} ${pi / 2} 0"/></joint>
     <link name="${prefix}_foot">
-      <visual><geometry><sphere radius="0.006"/></geometry><material name="black"/></visual>
       <collision><geometry><sphere radius="0.006"/></geometry></collision>
       <inertial><mass value="0.005"/><inertia ixx="7.2e-08" ixy="0" ixz="0" iyy="7.2e-08" iyz="0" izz="7.2e-08"/></inertial>

File: rumblex_description/urdf/nox_mesh.urdf.xacro (robot description, xacro)
@@ -5,8 +5,5 @@
   <xacro:include filename="$(find rumblex_description)/urdf/ros2_control.xacro"/>
   <xacro:property name="mesh_directory" value="package://rumblex_description/meshes/nox"/>
-  <xacro:property name="coxa_length" value="0.050"/>
-  <xacro:property name="femur_length" value="0.063"/>
-  <xacro:property name="tibia_length" value="0.099"/>
-  <xacro:property name="coxa_height" value="0.045"/>
+  <xacro:property name="coxa_height" value="0.0525"/>
   <xacro:arg name="use_sim" default="false"/>
   <xacro:if value="$(arg use_sim)">
@@ -15,27 +12,27 @@
   </xacro:if>
   <link name="base_link">
-    <visual><origin xyz="0 0 0"/><geometry><mesh filename="${mesh_directory}/assembly_torso_servo.stl" scale="0.001 0.001 0.001"/></geometry><material name="dark_gray"/></visual>
+    <visual><origin xyz="0 0 0"/><geometry><mesh filename="${mesh_directory}/assembly_body_servo.stl" scale="0.001 0.001 0.001"/></geometry><material name="dark_gray"/></visual>
     <collision><origin xyz="0 0 0.020"/><geometry><box size="0.240 0.180 0.025"/></geometry></collision>
     <inertial><origin xyz="0 0 0.045"/><mass value="0.80"/><inertia ixx="0.003" ixy="0" ixz="0" iyy="0.004" iyz="0" izz="0.005"/></inertial>
   </link>
-  <xacro:mesh_hexapod_leg prefix="right_front" cx="0.109" cy="0.068" psi_deg="45.0"/>
-  <xacro:mesh_hexapod_leg prefix="right_mid" cx="0.000" cy="0.088" psi_deg="90.0"/>
-  <xacro:mesh_hexapod_leg prefix="right_back" cx="-0.109" cy="0.068" psi_deg="135.0"/>
-  <xacro:mesh_hexapod_leg prefix="left_front" cx="0.109" cy="-0.068" psi_deg="-45.0"/>
-  <xacro:mesh_hexapod_leg prefix="left_mid" cx="0.000" cy="-0.088" psi_deg="-90.0"/>
-  <xacro:mesh_hexapod_leg prefix="left_back" cx="-0.109" cy="-0.068" psi_deg="-135.0"/>
-  <!-- Head transforms reproduce the zero-angle placement in
-       cad/assembly_complete.py.  The body mesh already contains the yaw
+  <xacro:mesh_hexapod_leg prefix="right_front" cx="0.114765879310439" cy="0.069765879310439" psi_deg="45.0"/>
+  <xacro:mesh_hexapod_leg prefix="right_mid" cx="0.000" cy="0.095175" psi_deg="90.0"/>
+  <xacro:mesh_hexapod_leg prefix="right_back" cx="-0.114765879310439" cy="0.069765879310439" psi_deg="135.0"/>
+  <xacro:mesh_hexapod_leg prefix="left_front" cx="0.114765879310439" cy="-0.069765879310439" psi_deg="-45.0"/>
+  <xacro:mesh_hexapod_leg prefix="left_mid" cx="0.000" cy="-0.095175" psi_deg="-90.0"/>
+  <xacro:mesh_hexapod_leg prefix="left_back" cx="-0.114765879310439" cy="-0.069765879310439" psi_deg="-135.0"/>
+  <!-- Head transforms reproduce the standing-pose placement in
+       cad/robot_nox/assembly_complete.py.  The body mesh already contains the yaw
        servo; these links add its coxa bracket and the pitch-mounted head. -->
   <joint name="head_yaw_joint" type="revolute">
     <parent link="base_link"/>
     <child link="head_yaw_link"/>
-    <origin xyz="0.140175 0 0.04825"/>
-    <axis xyz="0 0 -1"/>
+    <origin xyz="0.140175 0 0.0525" rpy="${pi} 0 0"/>
+    <axis xyz="0 0 1"/>
     <limit lower="${-30*pi/180}" upper="${30*pi/180}" effort="1.5" velocity="4.0"/>
   </joint>
   <link name="head_yaw_link">
     <visual>
-      <origin xyz="0.0295 0 -0.0143" rpy="${90*pi/180} 0 ${-90*pi/180}"/>
+      <origin xyz="0.0295 0 0.0185" rpy="${-pi/2} 0 ${pi/2}"/>
       <geometry><mesh filename="${mesh_directory}/assembly_coxa.stl" scale="0.001 0.001 0.001"/></geometry>
       <material name="dark_gray"/>
@@ -46,11 +43,11 @@
     <parent link="head_yaw_link"/>
     <child link="head_pitch_link"/>
-    <origin xyz="0.05313138535886 0.0143 -0.00338993770857"/>
-    <axis xyz="0 -1 0"/>
+    <origin xyz="0.053131385358869 -0.0185 0.0075064241990335" rpy="${pi/2} -1.5576858731134 ${-pi}"/>
+    <axis xyz="0 0 -1"/>
     <limit lower="${-20*pi/180}" upper="${20*pi/180}" effort="1.5" velocity="4.0"/>
   </joint>
   <link name="head_pitch_link">
     <visual>
-      <origin xyz="0 0 0.035" rpy="${180*pi/180} 0 0"/>
+      <origin xyz="-0.035 0 0.00425" rpy="${pi/2} 0 ${pi/2}"/>
       <geometry><mesh filename="${mesh_directory}/assembly_head.stl" scale="0.001 0.001 0.001"/></geometry>
       <material name="dark_gray"/>

Commit message: fix wrong femur behavior of the simulation

File: rumblex_description/urdf/mesh_leg.xacro (robot description, xacro)
@@ -4,6 +4,7 @@
        Joint frames are the horn mounting faces, not the simplified IK frames
        in leg.xacro. Zero pose matches assembly_complete: CAD angles 0/0/180.
-       Positive joint angles increase the CAD connection angles. The STL
-       exports already contain the femur and tibia rolls; do not apply again. -->
+       The femur axis follows the kinematics convention: positive angles lift
+       the leg, opposite to the CAD connection angle. The STL exports already
+       contain the femur and tibia rolls; do not apply again. -->
   <xacro:macro name="mesh_hexapod_leg" params="prefix cx cy psi_deg">
     <xacro:property name="mount_yaw" value="${psi_deg * pi / 180.0}"/>
@@ -28,5 +29,5 @@
     <joint name="${prefix}_femur_joint" type="revolute">
       <parent link="${prefix}_coxa_link"/><child link="${prefix}_femur_link"/>
-      <origin xyz="0.053131385358869 -0.0185 0.0075064241990335" rpy="${pi / 2} -0.51048832191678 ${pi}"/><axis xyz="0 0 -1"/>
+      <origin xyz="0.053131385358869 -0.0185 0.0075064241990335" rpy="${pi / 2} -0.51048832191678 ${pi}"/><axis xyz="0 0 1"/>
       <limit lower="${-30 * pi / 180}" upper="${90 * pi / 180}" effort="3.0" velocity="6.0"/>
       <dynamics damping="0.1" friction="0.05"/>

File: rumblex_description/urdf/nira_model.xacro (robot description, xacro)
@@ -58,5 +58,5 @@
                      mass="0.12" meshes="${meshes}" material="dark_gray"/>
     <xacro:nira_joint name="${prefix}_femur_joint" parent="${prefix}_coxa_link" child="${prefix}_femur_link"
-                      xyz="0.0531313853589 -0.0185 0.00750642419903" rpy="1.57079632679 -0.510488321917 3.14159265359" axis="0 0 -1" lower="-30" upper="90"/>
+                      xyz="0.0531313853589 -0.0185 0.00750642419903" rpy="1.57079632679 -0.510488321917 3.14159265359" axis="0 0 1" lower="-30" upper="90"/>
     <xacro:nira_link name="${prefix}_femur_link" mesh="assembly_femur"
                      xyz="-0.035 0 0.00425" rpy="1.57079632679 0 1.57079632679"
