Commit message: add meshes for nira

File: rumblex_description/urdf/nox_mesh.urdf.xacro (robot description, xacro)
@@ -15,5 +15,5 @@
   </xacro:if>
   <link name="base_link">
-    <visual><origin xyz="0 0 0"/><geometry><mesh filename="${mesh_directory}/assembly_body_servo.stl" scale="0.001 0.001 0.001"/></geometry><material name="dark_gray"/></visual>
+    <visual><origin xyz="0 0 0"/><geometry><mesh filename="${mesh_directory}/assembly_torso_servo.stl" scale="0.001 0.001 0.001"/></geometry><material name="dark_gray"/></visual>
     <collision><origin xyz="0 0 0.020"/><geometry><box size="0.240 0.180 0.025"/></geometry></collision>
     <inertial><origin xyz="0 0 0.045"/><mass value="0.80"/><inertia ixx="0.003" ixy="0" ixz="0" iyy="0.004" iyz="0" izz="0.005"/></inertial>

Commit message: add house map

File: rumblex_description/urdf/nox_mesh.urdf.xacro (robot description, xacro)
@@ -55,3 +55,11 @@
     <inertial><mass value="0.001"/><inertia ixx="1e-8" ixy="0" ixz="0" iyy="1e-8" iyz="0" izz="1e-8"/></inertial>
   </link>
+  <!-- Nominal beam origin at the midpoint of the two CAD lidar front faces.
+       CAD +X maps to head_pitch_link +Y through the visual's rotation. -->
+  <joint name="lidar_joint" type="fixed">
+    <parent link="head_pitch_link"/>
+    <child link="lidar_link"/>
+    <origin xyz="-0.020194 0.063636 0.018754" rpy="0 0 ${pi/2}"/>
+  </joint>
+  <link name="lidar_link"/>
 </robot>

Commit message: fix rviz

File: rumblex_description/urdf/nox_mesh.urdf.xacro (robot description, xacro)
@@ -16,4 +16,11 @@
     <inertial><origin xyz="0 0 0.045"/><mass value="0.80"/><inertia ixx="0.003" ixy="0" ixz="0" iyy="0.004" iyz="0" izz="0.005"/></inertial>
   </link>
+  <!-- Match the bottom-plate IMU mounting frame in the primitive Nox model. -->
+  <joint name="imu_joint" type="fixed">
+    <parent link="base_link"/>
+    <child link="imu_link"/>
+    <origin xyz="0 0 0.0075" rpy="0 0 0"/>
+  </joint>
+  <link name="imu_link"/>
   <xacro:mesh_hexapod_leg prefix="left_front" cx="0.114765879310439" cy="0.069765879310439" psi_deg="45.0"/>
   <xacro:mesh_hexapod_leg prefix="left_mid" cx="0.000" cy="0.095175" psi_deg="90.0"/>
